File: hardware/taptdoa_1.x.brd (EAGLE design)
At the start: 66 x 63.2 mm, 91 parts, among them J5 105017-0001, U1 SN74HCT245PWR, U2 AP2112K-3.3TRG1, U3 STM32F303RET6, Y1 8MHz

Commit message: fix minor drc
Routing:
- net N$2: track 30.3 -> 29.2 mm
- net N$22: track 27.6 -> 28.2 mm
Changed lines of the file:
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@@
 <via x="65.024" y="49.784" extent="1-16" drill="0.3302"/>
 <wire x1="32.015" y1="43.5578" x2="32.015" y2="41.413" width="0.254" layer="1"/>
-<wire x1="32.015" y1="41.413" x2="32.004" y2="41.402" width="0.254" layer="1"/>
 <via x="23.876" y="41.402" extent="1-16" drill="0.3302"/>
 <via x="31.242" y="14.986" extent="1-16" drill="0.35"/>
@@
 <via x="59.69" y="25.4" extent="1-16" drill="0.35"/>
 <via x="56.896" y="27.178" extent="1-16" drill="0.35"/>
-<via x="53.086" y="27.178" extent="1-16" drill="0.35"/>
-<via x="49.276" y="27.178" extent="1-16" drill="0.35"/>
+<via x="53.594" y="27.178" extent="1-16" drill="0.35"/>
+<via x="50.292" y="27.178" extent="1-16" drill="0.35"/>
 <via x="47.244" y="25.908" extent="1-16" drill="0.35"/>
 <via x="43.434" y="25.908" extent="1-16" drill="0.35"/>
@@
 <wire x1="12.28" y1="20.32" x2="12.28" y2="21.082" width="0.1524" layer="1"/>
 <wire x1="26.25" y1="21.59" x2="25.19" y2="20.53" width="0.1524" layer="1"/>
-<wire x1="25.19" y1="20.53" x2="24.8784" y2="20.2184" width="0.1524" layer="1"/>
 <wire x1="53.76" y1="21.082" x2="53.76" y2="19.05" width="0.1524" layer="1"/>
 <wire x1="40.132" y1="18.376" x2="51.4348125" y2="18.376" width="0.1524" layer="1"/>
@@
 <wire x1="10.0886" y1="25.3133125" x2="9.9546875" y2="25.1794" width="0.1524" layer="1"/>
 <wire x1="9.9546875" y1="25.1794" x2="8.89" y2="25.1794" width="0.1524" layer="1"/>
-<wire x1="8.89" y1="25.1794" x2="8.6653125" y2="25.1794" width="0.1524" layer="1"/>
-<wire x1="4.572" y1="27.94" x2="4.203" y2="27.94" width="0.1524" layer="1"/>
 <wire x1="4.203" y1="27.94" x2="5.1964" y2="26.9466" width="0.1524" layer="1"/>
 <wire x1="5.1964" y1="26.9466" x2="6.5697875" y2="26.9466" width="0.1524" layer="1"/>
 <wire x1="8.3369875" y1="25.1794" x2="8.89" y2="25.1794" width="0.1524" layer="1"/>
 <wire x1="6.5697875" y1="26.9466" x2="8.3369875" y2="25.1794" width="0.1524" layer="1"/>
-<wire x1="4.72158125" y1="27.94" x2="4.203" y2="27.94" width="0.1524" layer="1"/>
 <wire x1="4.203" y1="27.94" x2="5.03830625" y2="28.77530625" width="0.1524" layer="1"/>
 <wire x1="5.03830625" y1="28.77530625" x2="5.5682125" y2="28.77530625" width="0.1524" layer="1"/>
@@
 <wire x1="12.7" y1="25.4" x2="13.208" y2="25.4" width="0.1524" layer="16"/>
 <wire x1="13.208" y1="25.4" x2="13.4168" y2="25.6088" width="0.1524" layer="16"/>
-<wire x1="13.4168" y1="25.6088" x2="13.462" y2="25.6088" width="0.1524" layer="16"/>
 <wire x1="13.6817875" y1="25.6088" x2="13.97549375" y2="25.90250625" width="0.1524" layer="16"/>
 <wire x1="13.4168" y1="25.6088" x2="13.6817875" y2="25.6088" width="0.1524" layer="16"/>
@@
 <contactref element="D3" pad="C"/>
 <contactref element="R25" pad="2"/>
-<wire x1="10.414" y1="33.413" x2="15.24" y2="33.413" width="0.1524" layer="1"/>
 <via x="7.62" y="28.4706" extent="1-16" drill="0.35"/>
 <wire x1="7.62" y1="28.4706" x2="6.35" y2="27.2006" width="0.1524" layer="16"/>
@@
 <wire x1="7.62" y1="28.4706" x2="7.62" y2="30.3960375" width="0.1524" layer="1"/>
 <wire x1="7.62" y1="30.3960375" x2="9.1948" y2="31.9708375" width="0.1524" layer="1"/>
+<wire x1="9.1948" y1="32.1938" x2="9.1948" y2="31.9708375" width="0.1524" layer="1"/>
+<wire x1="15.24" y1="33.413" x2="10.414" y2="33.413" width="0.1524" layer="1"/>
+<wire x1="10.414" y1="33.413" x2="10.16" y2="33.159" width="0.1524" layer="1"/>
 <wire x1="9.1948" y1="31.9708375" x2="9.1948" y2="32.1938" width="0.1524" layer="1"/>
 <wire x1="9.1948" y1="32.1938" x2="10.16" y2="33.159" width="0.1524" layer="1"/>
-<wire x1="10.16" y1="33.159" x2="10.414" y2="33.413" width="0" layer="19" extent="1-1"/>
 </signal>
 </signals>
